File: DAQ-MCU.kicad_sch (KiCad schematic)
At the start: 14 parts, among them U8 STM32G474CEUx

Commit message: data ready signals
Parts:
- added R164: 33, Resistor_SMD:R_0603_1608Metric_Pad0.98x0.95mm_HandSolder, symbol Device:R
Connections:
- net at U8.29 (PC6): now also R164.1
- new net DATA_READY: R164.2
Changed lines of the file:
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@@
 	(wire
 		(pts
+			(xy 105.41 85.09) (xy 109.22 85.09)
+		)
+		(stroke
+			(width 0)
+			(type default)
+		)
+	)
+	(wire
+		(pts
 			(xy 30.48 31.75) (xy 43.18 31.75)
 		)
@@
 	(wire
 		(pts
-			(xy 111.76 82.55) (xy 123.19 82.55)
+			(xy 105.41 82.55) (xy 123.19 82.55)
 		)
 		(stroke
@@
 	(wire
 		(pts
+			(xy 116.84 85.09) (xy 123.19 85.09)
+		)
+		(stroke
+			(width 0)
+			(type default)
+		)
+	)
+	(wire
+		(pts
 			(xy 92.71 33.02) (xy 92.71 31.75)
 		)
@@
 		)
 	)
+	(hierarchical_label "DATA_READY"
+		(shape output)
+		(at 105.41 85.09 180)
+		(fields_autoplaced yes)
+		(effects
+			(font
+				(size 1.27 1.27)
+			)
+			(justify right)
+		)
+	)
 	(hierarchical_label "SPI1_MISO"
 		(shape output)
@@
 	(hierarchical_label "SPI1_CS"
 		(shape input)
-		(at 111.76 82.55 180)
+		(at 105.41 82.55 180)
 		(fields_autoplaced yes)
 		(effects
@@
 					(unit 1)
 				)
+			)
+		)
+	)
+	(symbol
+		(lib_id "Device:R")
+		(at 113.03 85.09 270)
+		(mirror x)
+		(unit 1)
+		(exclude_from_sim no)
+		(in_bom yes)
+		(on_board yes)
+		(dnp no)
+		(property "Reference" "R164"
+			(at 118.364 84.074 90)
+			(effects
+				(font
+					(size 1.27 1.27)
+				)
+			)
+		)
+		(property "Value" "33"
+			(at 113.03 85.09 90)
+			(effects
+				(font
+					(size 1.27 1.27)
+				)
+			)
+		)
+		(property "Footprint" "Resistor_SMD:R_0603_1608Metric_Pad0.98x0.95mm_HandSolder"
+			(at 113.03 86.868 90)
+			(effects
+				(font
+					(size 1.27 1.27)
+				)
+				(hide yes)
+			)
+		)
+		(property "Datasheet" "~"
+			(at 113.03 85.09 0)
+			(effects
+				(font
+					(size 1.27 1.27)
+				)
+				(hide yes)
+			)
+		)
+		(property "Description" "Resistor"
+			(at 113.03 85.09 0)
+			(effects
+				(font
+					(size 1.27 1.27)
+				)
+				(hide yes)
+			)
+		)
+		(pin "2"
+		)
+		(pin "1"
+		)
+		(instances
+			(project "ELS-overall_schematic"
+				(path "/e163ac89-2584-465c-83de-a2d940380c99/5cd54913-de05-4d24-857a-a5c68b00a6b8"
+					(reference "R164")
+					(unit 1)
+				)
+				(path "/e163ac89-2584-465c-83de-a2d940380c99/e4b9ffc8-077d-4e5f-a588-3fe86cc1b2b4"
+					(reference "R165")
+					(unit 1)
+				)
+				(path "/e163ac89-2584-465c-83de-a2d940380c99/55ac26b6-e7af-4ca8-92b1-4cb6fa926089"
+					(reference "R166")
+					(unit 1)
+				)
+				(path "/e163ac89-2584-465c-83de-a2d940380c99/3ba2c326-b309-4f85-817b-a64327d92b06"
+					(reference "R167")
+					(unit 1)
+				)

Commit message: gnd and gnda
Parts:
- removed R24: 10K, Resistor_SMD:R_0603_1608Metric_Pad0.98x0.95mm_HandSolder, symbol Device:R
- added C172: 100n, symbol Device:C
- added D13: D_Schottky, symbol Device:D_Schottky
- added D14: ESDA6V1-5SC6, Package_TO_SOT_SMD:SOT-23-6, symbol Power_Protection:ESDA6V1-5SC6
Connections:
- net GND: now also C172.2, D14.2 (GND)
- net NRST: now also C172.1, D14.4 (IO3)
- net SYS_SWCLK: now also D14.6 (IO5)
- net SYS_SWDIO: now also D14.5 (IO4)
- net USART2_RX: now also D14.1 (IO1)
- net USART2_TX: now also D14.3 (IO2)
- net VDD: no longer J_A2.1 (Pin_1)
- new net: D13.2 (A), J_A2.1 (Pin_1)
- new net +5V: D13.1 (K)
