File: FEE-Si.kicad_sch (KiCad schematic)
At the start: 36 parts, among them J4 Conn_01x02_Pin, U11 OPA2356-Q1, U12 OPA2356-Q1

Commit message: gnd and gnda
Connections:
- net GND: no longer R49.1, TH1.2, TH2.2, U13.14 (REF-)
- net GNDA: now also R49.1, TH1.2, TH2.2, U13.14 (REF-)
Changed lines of the file:
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@@
+	)
+	(symbol
+		(lib_id "power:GNDA")
+		(at 39.37 171.45 0)
+		(unit 1)
+		(exclude_from_sim no)
+		(in_bom yes)
+		(on_board yes)
+		(dnp no)
+		(fields_autoplaced yes)
+		(property "Reference" "#PWR0112"
+			(at 39.37 177.8 0)
+			(effects
+				(font
+					(size 1.27 1.27)
+				)
+				(hide yes)
+			)
+		)
+		(property "Value" "GNDA"
+			(at 39.37 176.53 0)
+			(effects
+				(font
+					(size 1.27 1.27)
+				)
+			)
+		)
+		(property "Footprint" ""
+			(at 39.37 171.45 0)
+			(effects
+				(font
+					(size 1.27 1.27)
+				)
+				(hide yes)
+			)
+		)
+		(property "Datasheet" ""
+			(at 39.37 171.45 0)
+			(effects
+				(font
+					(size 1.27 1.27)
+				)
+				(hide yes)
+			)
+		)
+		(property "Description" "Power symbol creates a global label with name \"GNDA\" , analog ground"
+			(at 39.37 171.45 0)
+			(effects
+				(font
+					(size 1.27 1.27)
+				)
+				(hide yes)
+			)
+		)
+		(pin "1"
+		)
+		(instances
+			(project "ELS-overall_schematic"
+				(path "/e163ac89-2584-465c-83de-a2d940380c99/e4b8c048-c621-4d07-8631-fadd488b1079"
+					(reference "#PWR0112")
+					(unit 1)
+				)
+				(path "/e163ac89-2584-465c-83de-a2d940380c99/3c02ebdb-ab1d-445f-8248-bb4b1800e421"
+					(reference "#PWR0170")
+					(unit 1)
+				)
+			)
+		)
 	)
 	(symbol
@@
 		(on_board yes)
 		(dnp no)
-		(fields_autoplaced yes)
 		(property "Reference" "#PWR0110"
 			(at 74.93 170.18 0)
@@
 			)
 		)
-		(property "Value" "GND"
-			(at 74.93 168.91 0)
-			(effects
-				(font
-					(size 1.27 1.27)
-				)
+		(property "Value" "GNDA"
+			(at 72.39 168.91 0)
+			(effects
+				(font
+					(size 1.27 1.27)
+				)
+				(justify left)
 			)
 		)
@@
 					(unit 1)
 				)
-			)
-		)
-	)
-	(symbol
-		(lib_id "power:GND")
-		(at 39.37 171.45 0)
-		(unit 1)
-		(exclude_from_sim no)
-		(in_bom yes)
-		(on_board yes)
-		(dnp no)
-		(fields_autoplaced yes)
-		(property "Reference" "#PWR0112"
-			(at 39.37 177.8 0)
-			(effects
-				(font
-					(size 1.27 1.27)
-				)
-				(hide yes)
-			)
-		)
-		(property "Value" "GND"
-			(at 39.37 176.53 0)
-			(effects
-				(font
-					(size 1.27 1.27)
-				)
-			)
-		)
-		(property "Footprint" ""
-			(at 39.37 171.45 0)
-			(effects
-				(font
-					(size 1.27 1.27)
-				)
-				(hide yes)
-			)
-		)
-		(property "Datasheet" ""
-			(at 39.37 171.45 0)
-			(effects
-				(font
-					(size 1.27 1.27)
-				)
-				(hide yes)
-			)
-		)
-		(property "Description" "Power symbol creates a global label with name \"GND\" , ground"
-			(at 39.37 171.45 0)
-			(effects
-				(font
-					(size 1.27 1.27)
-				)
-				(hide yes)
-			)
-		)
-		(pin "1"
-		)
-		(instances
-			(project "ELS-overall_schematic"
-				(path "/e163ac89-2584-465c-83de-a2d940380c99/e4b8c048-c621-4d07-8631-fadd488b1079"
-					(reference "#PWR0112")
-					(unit 1)
-				)
-				(path "/e163ac89-2584-465c-83de-a2d940380c99/3c02ebdb-ab1d-445f-8248-bb4b1800e421"
-					(reference "#PWR0170")
-					(unit 1)
-				)
